Commit message: Add files via upload
add gazebo launch file, add yaml file for joint velocity control, fix urdf model

File: rover_project/rover_description/urdf/rover.urdf (robot description, URDF)
Before this commit: robot Rover Platform, 5 links, 4 joints
Links:
- link base_link: mass 5 -> None
Joints:
- removed joint left_wheel_holder_to_left_wheel
- removed joint right_wheel_holder_to_right_wheel
- added joint holder2wheel_left: type continuous, parent left_wheel_holder_link, child left_wheel_link, origin xyz=-0.15 0 -0.1 rpy=0 -1.57075 0, axis 0 0 1
- added joint holder2wheel_right: type continuous, parent right_wheel_holder_link, child right_wheel_link, origin xyz=0.15 0 -0.1 rpy=0 1.57075 0, axis 0 0 1
- joint base_to_left_wheel_holder: origin xyz=-0.4 0.2 -0.2 rpy=0 0 0 -> xyz=-0.4 0.2 -0.1 rpy=0 0 0
- joint base_to_right_wheel_holder: origin xyz=0.4 0.2 -0.2 rpy=0 0 0 -> xyz=0.4 0.2 -0.1 rpy=0 0 0

Commit message: Add files via upload
Add caster to urdf model

File: rover_project/rover_description/urdf/rover.urdf (robot description, URDF)
Before this commit: robot Rover Platform, 5 links, 4 joints
Links:
- added link caster_link, mass 0.5; collision sphere radius=0.2; visual sphere radius=0.2
- added link dummy_link
- link base_link: mass None -> 5; geometry collision box size=1.0 1.0 0.2; visual box size=1.0 1. 0.2
Joints:
- removed joint base_to_left_wheel_holder
- removed joint base_to_right_wheel_holder
- added joint base2caster: type fixed, parent base_link, child caster_link, origin xyz=0 -0.25 -0.1 rpy=0 0 0, axis 0 0 1
- added joint base2holder_left: type fixed, parent base_link, child left_wheel_holder_link, origin xyz=-0.4 0.3 -0.1 rpy=0 0 0
- added joint base2holder_right: type fixed, parent base_link, child right_wheel_holder_link, origin xyz=0.4 0.3 -0.1 rpy=0 0 0
- added joint dummy_joint: type fixed, parent dummy_link, child base_link

Commit message: Add files via upload
Correctly find the pose of the rover. Implemented the control algorithm (without testing).

File: rover_project/rover_description/urdf/rover.urdf (robot description, URDF)
Before this commit: robot Rover Platform, 7 links, 6 joints
Links:
- removed link caster_link
- added link caster, mass 0.5; collision box size=0.1 0.2 0.3; visual box size=0.1 0.2 0.3
Joints:
- joint base2caster: child caster_link -> caster; origin xyz=0 -0.25 -0.1 rpy=0 0 0 -> xyz=0 -0.4 -0.1 rpy=0 0 0

Commit message: Add files via upload
tested control algorithm, fixed calculation of yaw data

File: rover_project/rover_description/urdf/rover.urdf (robot description, URDF)
Before this commit: robot Rover Platform, 7 links, 6 joints
Joints:
- joint dummy_joint: origin (none) -> xyz=0 -0.3 0.2 rpy=0 0 0

Commit message: update rover description

File: rover_project/rover_description/urdf/rover.urdf (robot description, URDF)
Before this commit: robot Rover Platform, 7 links, 6 joints
Links:
- removed link caster
- removed link left_wheel_holder_link
- removed link left_wheel_link
- removed link right_wheel_holder_link
- removed link right_wheel_link
- link base_link: geometry collision box size=0.16 0.16 0.004; visual box size=0.16 0.16 0.004
Joints:
- removed joint base2caster
- removed joint base2holder_left
- removed joint base2holder_right
- removed joint holder2wheel_left
- removed joint holder2wheel_right
- joint dummy_joint: origin xyz=0 -0.3 0.2 rpy=0 0 0 -> xyz=0 -0.055 0.002 rpy=0 0 0
